File: Eagle/Powerstep_communication/task_eagle.sch (EAGLE design)
At the start: 104 parts, among them IC2 ATMEGA640-16AI, IC3 74ACT125D, IC7 FT232RL, IC8 MAX485, K1 G5LE, K2 G5LE, K3 G5LE, K6 G5LE, U1 TC1262-33VDB, U2 Tyco 5-6605758-1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

Commit message: powerstep board
Parts:
- removed ANALOG_IN, X2: (no value), con-molex:KK-156-4
- added ANALOG_ADC: (no value), con-molex:KK-156-4
- added SW1: (no value), special:SW_DIP-4
- C16: value 100nF -> 0.1nF
- R22, R25, R28: value 12K -> 1K
Connections:
- removed net +5V: C15.1, F1.1
- removed net A1_12V: ANALOG_IN-1.S
- removed net A2_12V: ANALOG_IN-2.S
- removed net A3_12V: ANALOG_IN-3.S
- removed net A4_12V: ANALOG_IN-4.S
- new net N$4: SW1.1, SW1.2, SW1.3, SW1.4, U$1.ADDR
- net A0_ADC: now also ANALOG_ADC-1.S; no longer IC2.(ADC4/TCK)PF4, X2-1.S
- net A1_ADC: now also ANALOG_ADC-2.S; no longer IC2.(ADC5/TMS)PF5, X2-2.S
- net A2_ADC: now also ANALOG_ADC-3.S; no longer IC2.(ADC6/TDO)PF6, X2-3.S
- net A3_ADC: now also ANALOG_ADC-4.S; no longer IC2.(ADC7/TDI)PF7, X2-4.S
- net GND: now also SW1.8
- net SCL_ADC: now also SW1.6
- net SDA_ADC: now also SW1.5
- net VCC: now also C15.1, F1.1, SW1.7

Commit message: eagle powerstepproto
Parts:
- removed ANALOG_ADC, DIGITAL_IN1: (no value), con-molex:KK-156-4
- removed MAIN_INPUT, SERIAL, X1: (no value), con-molex:KK-156-2
- removed X3: (no value), con-molex:KK-156-8
- added DIGITAL_INPUT: (no value), SparkFun-Connectors:CONN_04
- added J1, J2: (no value), SparkFun-Connectors:CONN_02
- added J4: (no value), SparkFun-Connectors:CONN_10"
- added RELAY_I/O: (no value), SparkFun-Connectors:CONN_08"
Connections:
- new net N$19: J4.1, U$2.A+
- new net N$33: J4.2, U$2.B+
- new net N$34: J4.5, U$2.B-
- new net N$35: J4.6, U$2.A-
- net 12V_IN: now also J2.2; no longer MAIN_INPUT-2.S
- net A: now also J1.1; no longer SERIAL-1.S
- net A0_ADC: now also J4.7; no longer ANALOG_ADC-1.S
- net A1_ADC: now also J4.8; no longer ANALOG_ADC-2.S
- net A2_ADC: now also J4.9; no longer ANALOG_ADC-3.S
- net A3_ADC: now also J4.10; no longer ANALOG_ADC-4.S
- net B: now also J1.2; no longer SERIAL-2.S
- net COMM_1: now also RELAY_I/O.1; no longer X3-1.S
- net COMM_2: now also RELAY_I/O.2; no longer X3-2.S
- net COMM_3: now also RELAY_I/O.3; no longer X3-3.S
- net COMM_4: now also RELAY_I/O.4; no longer X3-4.S
- net DIG1_48V: now also RELAY_I/O.5; no longer X3-5.S
- net DIG2_48V: now also RELAY_I/O.6; no longer X3-6.S
- net DIG3_48V: now also RELAY_I/O.7; no longer X3-7.S
- net DIG4_48V: now also RELAY_I/O.8; no longer X3-8.S
- net DIG_24V_IN_1: now also DIGITAL_INPUT.1; no longer DIGITAL_IN1-1.S
- net DIG_24V_IN_2: now also DIGITAL_INPUT.2; no longer DIGITAL_IN1-2.S
- net DIG_24V_IN_3: now also DIGITAL_INPUT.3; no longer DIGITAL_IN1-3.S
- net DIG_24V_IN_4: now also DIGITAL_INPUT.4; no longer DIGITAL_IN1-4.S
- net GND: now also J2.1, J4.3; no longer MAIN_INPUT-1.S, X1-1.S
- net RESET_1: now also IC2.PJ0(RXD3/PCINT9); no longer IC2.(OC1A/PCINT5)PB5
- net RESET_FTDI: now also IC2.(OC3A/AIN1)PE3; no longer IC2.(A15)PC7
- net RX_FTDI: now also IC2.(RXD0/PCIN8)PE0; no longer IC2.PJ0(RXD3/PCINT9)
- net TX_FTDI: now also IC2.(TXD0)PE1; no longer IC2.PJ1(TXD3/PCINT10)
- net VMOT: now also J4.4; no longer X1-2.S
Other:
- note removed: "12V"
- note removed: "GND"

Commit message: powerstep.brd
Parts:
- removed DIGITAL_INPUT: (no value), SparkFun-Connectors:CONN_04
- removed J1, J2: (no value), SparkFun-Connectors:CONN_02
- removed J4: (no value), SparkFun-Connectors:CONN_10"
- removed RELAY_I/O: (no value), SparkFun-Connectors:CONN_08"
- added U$4: 10_R44 - 1821326, Pheonix_connectors:10_R44 - 1821326
- added U$5: 16_R56 - 1821384, Pheonix_connectors:16_R56 - 1821384
- C1, C2, C3: value 100uF -> 100u
Connections:
- removed net 12V_INPUT: OC1A.A, OC1B.A, OC1C.A, OC1D.A
- removed net N$19: J4.1, U$2.A+
- removed net N$33: J4.2, U$2.B+
- removed net N$34: J4.5, U$2.B-
- removed net N$35: J4.6, U$2.A-
- new net A+_STEP: U$2.A+, U$5.P$3
- new net A-_STEP: U$2.A-, U$5.P$8
- new net B+_STEP: U$2.B+, U$5.P$4
- new net B-_STEP: U$2.B-, U$5.P$7
- net 12V: now also OC1A.A, OC1B.A, OC1C.A, OC1D.A
- net 12V_IN: now also U$4.P$9; no longer J2.2
- net A: now also U$5.P$1; no longer J1.1
- net A0_ADC: now also U$5.P$9; no longer J4.7
- net A1_ADC: now also U$5.P$10; no longer J4.8
- net A2_ADC: now also U$5.P$11; no longer J4.9
- net A3_ADC: now also U$5.P$12; no longer J4.10
- net B: now also U$5.P$2; no longer J1.2
- net COMM_1: now also U$4.P$8; no longer RELAY_I/O.1
- net COMM_2: now also U$4.P$7; no longer RELAY_I/O.2
- net COMM_3: now also U$4.P$6; no longer RELAY_I/O.3
- net COMM_4: now also U$4.P$5; no longer RELAY_I/O.4
- net DIG1_48V: now also U$4.P$4; no longer RELAY_I/O.5
- net DIG2_48V: now also U$4.P$3; no longer RELAY_I/O.6
- net DIG3_48V: now also U$4.P$2; no longer RELAY_I/O.7
- net DIG4_48V: now also U$4.P$1; no longer RELAY_I/O.8
- net DIG_24V_IN_1: now also U$5.P$13; no longer DIGITAL_INPUT.1
- net DIG_24V_IN_2: now also U$5.P$14; no longer DIGITAL_INPUT.2
- net DIG_24V_IN_3: now also U$5.P$15; no longer DIGITAL_INPUT.3
- net DIG_24V_IN_4: now also U$5.P$16; no longer DIGITAL_INPUT.4
- net GND: now also U$4.P$10, U$5.P$5; no longer J2.1, J4.3
- net VMOT: now also U$5.P$6; no longer J4.4
Other:
- note removed: "COMM_1"
- note removed: "COMM_2"
- note removed: "COMM_3"
- note removed: "COMM_4"
- note removed: "DIG1_48V"
- note removed: "DIG2_48V"
- note removed: "DIG3_48V"
- note removed: "DIG4_48V"
