File: Eagle/power_multiIO/task_eagle.sch (EAGLE design)
At the start: 100 parts, among them IC2 ATMEGA640-16AI, IC3 74ACT125D, IC7 FT232RL, IC8 MAX485, K1 G5LE, K2 G5LE, K3 G5LE, K6 G5LE, U1 TC1262-33VDB, U2 Tyco 5-6605758-1, U3 ENC28J60-SSOP, Y1 RESONATORMU, Y2 25MHz

Commit message: rfid and power_multiIO
Parts:
- added ADJUST_OVLO: 200K, SmartPrj:R-EU_R0603
- added ADJUST_UVLO: 250K, SmartPrj:R-EU_R0603
- added C17: 0.47uF, SmartPrj:C-EU0603-RND
- added C18: 4.7uF, SmartPrj:C-EU0603-RND
- added C21: 0.1uF, SmartPrj:C-EU0603-RND
- added PWR-LED1: Amber, SparkFun:LED0603
- added R15_BYPASS8: 0R, SmartPrj:R-EU_R0603
- added R26, R27: 2.2M, SmartPrj:R-EU_R0603
- added R38: 2.74K, SmartPrj:R-EU_R0603
- added R39, R40, R41: 100K, SmartPrj:R-EU_R0603
- added R42, R43: 10K, SmartPrj:R-EU_R0603
- added U$37: MAX14571, MAX14571:MAX14571
- added U$38: STPS5L60S, STPS5L60S:STPS5L60S
- added U$39: SM6T36CA, ref-packages:SM6T36CA
- added U$40: NC7WZ07P6X, ref-packages:NC7WZ07P6X
- added U$41, U$42: EEV-FK1H331Q, EEVFK1H331Q:EEV-FK1H331Q
- C1, C2, C3: value 100uF -> 100u
Connections:
- new net 12V_FET: C17.1, D3.C, PFET-M.S, R26.1, R27.1, U$37.IN@1, U$37.IN@2, U$37.IN@3, U$39.P$2
- new net N$40: PWR-LED1.A, R43.1
- new net N$45: PWR-LED1.C, U$40.Y1
- new net N$46: R39.1, U$40.A2
- new net N$55: R15_BYPASS8.2, U$40.Y2
- new net OVLO: ADJUST_OVLO.1, R26.2, U$37.OVLO
- new net SETI: R38.1, U$37.SETI
- new net UVLO: ADJUST_UVLO.1, R27.2, U$37.UVLO
- new net XX: R42.2, U$37.FLAG, U$40.A1
- net 12V: now also C18.1, U$37.OUT@1, U$37.OUT@2, U$37.OUT@3, U$38.P$2, U$41.P$1, U$42.P$1; no longer D3.C, PFET-M.S
- net GND: now also ADJUST_OVLO.2, ADJUST_UVLO.2, C17.2, C18.2, C21.2, R38.2, R39.2, R40.1, R41.1, U$37.GND, U$37.HVEN, U$38.P$1, U$39.P$1, U$40.GND, U$41.P$2, U$42.P$2
- net VCC: now also C21.1, R15_BYPASS8.1, R40.2, R41.2, R42.1, R43.2, U$37.EN, U$37.RIEN, U$40.VCC
Other:
- note added: "OVER AND UNDER VOLTAGE"
- note added: "Protection circuit"
- note added: "SET CURRENT"
