File: Eagle/power_multiIO/task_eagle.brd (EAGLE design)
At the start: 85 x 123.9 mm, 100 parts, among them IC2 ATMEGA640-16AI, IC3 74ACT125D, IC7 FT232RL, IC8 MAX485, K1 G5LE, K2 G5LE, K3 G5LE, K6 G5LE, U1 TC1262-33VDB, U2 Tyco 5-6605758-1, U3 ENC28J60-SSOP, Y2 25MHz

Commit message: rfid and power_multiIO
Parts:
- added ADJUST_OVLO: 200K, SmartPrj:R0603-ROUND
- added ADJUST_UVLO: 250K, SmartPrj:R0603-ROUND
- added C17: 0.47uF, SmartPrj:C0603-ROUND
- added C18: 4.7uF, SmartPrj:C0603-ROUND
- added C21: 0.1uF, SmartPrj:C0603-ROUND
- added PWR-LED1: Amber, SparkFun:LED-0603
- added R15_BYPASS8: 0R, SmartPrj:R0603-ROUND
- added R26, R27: 2.2M, SmartPrj:R0603-ROUND
- added R38: 2.74K, SmartPrj:R0603-ROUND
- added R39, R40, R41: 100K, SmartPrj:R0603-ROUND
- added R42, R43: 10K, SmartPrj:R0603-ROUND
- added U$37: MAX14571, MAX14571:TSSOP14
- added U$38: STPS5L60S, STPS5L60S:SMC
- added U$39: SM6T36CA, ref-packages:DO214AA
- added U$40: NC7WZ07P6X, ref-packages:SC70-6L
- added U$41, U$42: EEV-FK1H331Q, EEVFK1H331Q:EEVFK1H331Q
- moved C12 23.3 mm to (58.5, 88.8), flipped to the bottom
- moved DC2DC_1 18.3 mm to (54.2, 93.5), turned to 0 degrees
- moved D3 16.5 mm to (58.5, 105.1)
- moved PFET-M 16.1 mm to (62.9, 108.3)
- moved U$4 15.0 mm to (80.4, 103.8)
- moved K1 14.8 mm to (60.5, 126.2)
- moved K2 14.8 mm to (26.1, 126.2)
- moved K3 14.8 mm to (8.84, 126.3)
- moved K6 14.8 mm to (43.3, 126.2)
- moved U$5 3.79 mm to (80.6, 38.8)
Connections:
- new net 12V_FET: C17.1, D3.C, PFET-M.3, R26.1, R27.1, U$37.IN@1, U$37.IN@2, U$37.IN@3, U$39.C
- new net N$40: PWR-LED1.A, R43.1
- new net N$45: PWR-LED1.C, U$40.5
- new net N$46: R39.1, U$40.2
- new net N$55: R15_BYPASS8.2, U$40.6
- new net OVLO: ADJUST_OVLO.1, R26.2, U$37.OVLO
- new net SETI: R38.1, U$37.SETI
- new net UVLO: ADJUST_UVLO.1, R27.2, U$37.UVLO
- new net XX: R42.2, U$37.FLAG, U$40.1
- net 12V: now also C18.1, U$37.OUT@1, U$37.OUT@2, U$37.OUT@3, U$38.1, U$41.P$2, U$42.P$2; no longer D3.C, PFET-M.3
- net GND: now also ADJUST_OVLO.2, ADJUST_UVLO.2, C17.2, C18.2, C21.2, R38.2, R39.2, R40.1, R41.1, U$37.GND, U$37.HVEN, U$38.2, U$39.A, U$40.3, U$41.P$1, U$42.P$1
- net VCC: now also C21.1, R15_BYPASS8.1, R40.2, R41.2, R42.1, R43.2, U$37.EN, U$37.RIEN, U$40.4
Routing:
- net GND: track 733.7 -> 839.3 mm
- net 12V: track 54.3 -> 123.6 mm, vias 0 -> 2
- net VCC: track 413.0 -> 463.3 mm, vias 22 -> 25
- net 12V_FET: track 0.00 -> 26.4 mm, vias 0 -> 1
- net RELAY_3_IN: track 77.0 -> 92.8 mm
- net RELAY_4_IN: track 85.4 -> 100.3 mm
- net RELAY_2_IN: track 63.5 -> 78.5 mm
- net RELAY_1_IN: track 67.8 -> 82.6 mm, vias 1 -> 3
- net SETI: track 0.00 -> 11.2 mm
- net XX: track 0.00 -> 8.22 mm
- net OVLO: track 0.00 -> 8.01 mm
- net 12V_IN: track 29.9 -> 22.3 mm
- net UVLO: track 0.00 -> 4.16 mm
- net A0_ADC: track 13.1 -> 10.5 mm, vias 0 -> 1
- net N$55: track 0.00 -> 2.43 mm
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Other:
- board size 85 x 123.9 mm -> 85 x 140.3 mm

Commit message: small hopper
Routing:
- net RELAY_4_IN: track 100.3 -> 87.4 mm
- net GND: track 839.3 -> 849.0 mm
- net RELAY_3_IN: track 92.8 -> 83.6 mm
- net CCW: track 79.8 -> 76.5 mm, vias 3 -> 2
Changed lines of the file:
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@@
 <wire x1="43.24858125" y1="72.42048125" x2="43.24858125" y2="70.17511875" width="0.6096" layer="1"/>
 <wire x1="43.24858125" y1="72.42048125" x2="43.24858125" y2="73.665078125" width="0.6096" layer="1"/>
-<wire x1="43.24858125" y1="73.665078125" x2="42.555159375" y2="74.3585" width="0.6096" layer="1"/>
-<wire x1="42.555159375" y1="74.3585" x2="41.14555625" y2="74.3585" width="0.6096" layer="1"/>
-<wire x1="41.14555625" y1="74.3585" x2="41.13861875" y2="74.3515625" width="0.6096" layer="1"/>
+<wire x1="43.24858125" y1="73.665078125" x2="42.56278125" y2="74.350878125" width="0.6096" layer="1"/>
+<wire x1="42.56278125" y1="74.350878125" x2="41.1379375" y2="74.350878125" width="0.6096" layer="1"/>
+<wire x1="41.1379375" y1="74.350878125" x2="41.13861875" y2="74.3515625" width="0.6096" layer="1"/>
 <wire x1="41.13861875" y1="69.2715625" x2="42.345025" y2="69.2715625" width="0.6096" layer="1"/>
 <wire x1="42.345025" y1="69.2715625" x2="43.24858125" y2="70.17511875" width="0.6096" layer="1"/>
@@
 <wire x1="54.0512" y1="52.3748" x2="54.0399" y2="52.385503125" width="0.254" layer="1"/>
 <wire x1="63.0936" y1="58.8772" x2="63.038059375" y2="58.93935625" width="0.254" layer="1"/>
-<wire x1="31.41218125" y1="74.4347" x2="40.8432" y2="74.422" width="0.6096" layer="1"/>
-<wire x1="28.4607" y1="77.383640625" x2="31.41218125" y2="74.4347" width="0.6096" layer="1"/>
+<wire x1="31.478221875" y1="74.361040625" x2="40.8432" y2="74.348340625" width="0.6096" layer="1"/>
+<wire x1="28.4607" y1="77.383640625" x2="31.478221875" y2="74.361040625" width="0.6096" layer="1"/>
 <wire x1="28.4607" y1="77.383640625" x2="28.460525" y2="79.15101875" width="0.6096" layer="1"/>
-<wire x1="40.8432" y1="74.422" x2="41.13861875" y2="74.3515625" width="0.254" layer="1"/>
+<wire x1="40.8432" y1="74.348340625" x2="41.13861875" y2="74.3515625" width="0.254" layer="1"/>
 <wire x1="11.9888" y1="54.2036" x2="11.9888" y2="52.9844" width="0.6096" layer="1"/>
 <wire x1="11.9888" y1="52.9844" x2="11.9994375" y2="52.983040625" width="0.254" layer="1"/>
@@
 <wire x1="56.771540625" y1="61.02858125" x2="60.944759375" y2="65.2018" width="0.6096" layer="1"/>
 <wire x1="60.944759375" y1="65.2018" x2="62.918340625" y2="65.2018" width="0.6096" layer="1"/>
-<wire x1="62.918340625" y1="65.2018" x2="63.731140625" y2="64.389" width="0.6096" layer="1"/>
+<wire x1="63.488571875" y1="64.63156875" x2="62.918340625" y2="65.2018" width="0.6096" layer="1"/>
+<wire x1="63.488571875" y1="64.63156875" x2="63.731140625" y2="64.389" width="0.6096" layer="1"/>
 <wire x1="63.731140625" y1="64.389" x2="63.731140625" y2="59.6324375" width="0.6096" layer="1"/>
 <wire x1="63.731140625" y1="59.6324375" x2="63.038059375" y2="58.93935625" width="0.6096" layer="1"/>
@@
 <wire x1="44.71161875" y1="104.38891875" x2="44.422053125" y2="104.38891875" width="0.3048" layer="16"/>
 <wire x1="44.422053125" y1="104.38891875" x2="43.47209375" y2="105.338878125" width="0.3048" layer="16"/>
+<wire x1="60.99321875" y1="71.0677375" x2="60.33115625" y2="71.0677375" width="0.254" layer="1"/>
+<wire x1="60.33115625" y1="71.0677375" x2="60.0202" y2="70.75678125" width="0.254" layer="1"/>
+<wire x1="60.0202" y1="70.75678125" x2="60.0202" y2="69.7585625" width="0.254" layer="1"/>
+<wire x1="60.0202" y1="69.7585625" x2="60.40628125" y2="69.37248125" width="0.254" layer="1"/>
+<wire x1="60.40628125" y1="69.37248125" x2="62.1309375" y2="69.37248125" width="0.254" layer="1"/>
+<wire x1="62.1309375" y1="69.37248125" x2="63.535559375" y2="67.967859375" width="0.254" layer="1"/>
+<wire x1="63.535559375" y1="67.967859375" x2="63.535559375" y2="64.67855625" width="0.254" layer="1"/>
+<wire x1="63.535559375" y1="64.67855625" x2="63.488571875" y2="64.63156875" width="0.254" layer="1"/>
 <wire x1="55.427325" y1="58.9348875" x2="55.4736" y2="58.9788" width="0" layer="19" extent="1-1"/>
-<wire x1="60.99321875" y1="71.0677375" x2="60.944759375" y2="65.2018" width="0" layer="19" extent="1-1"/>
 </signal>
 <signal name="TX_MAX">
@@
 <wire x1="46.321978125" y1="68.706996875" x2="46.332140625" y2="66.27368125" width="0.6096" layer="1"/>
 <wire x1="46.3169" y1="72.0699625" x2="46.327059375" y2="70.99808125" width="0.6096" layer="1"/>
-<wire x1="48.2871375" y1="73.03008125" x2="48.33861875" y2="73.0815625" width="0" layer="19" extent="1-16"/>
 <wire x1="46.76071875" y1="70.5415625" x2="46.327059375" y2="70.99808125" width="0.6096" layer="1"/>
 <wire x1="46.994396875" y1="68.0015625" x2="46.321978125" y2="68.706996875" width="0.6096" layer="1"/>
@@
 <wire x1="43.11141875" y1="80.1217625" x2="45.590459375" y2="80.1217625" width="0.254" layer="16"/>
 <via x="45.590459375" y="80.1217625" extent="1-16" drill="0.254"/>
-<wire x1="45.590459375" y1="80.1217625" x2="48.719740625" y2="83.26628125" width="0.254" layer="1"/>
-<wire x1="48.719740625" y1="83.26628125" x2="48.719740625" y2="85.747859375" width="0.254" layer="1"/>
-<via x="48.719740625" y="85.747859375" extent="1-16" drill="0.254"/>
-<wire x1="48.719740625" y1="85.747859375" x2="50.575084375" y2="85.747859375" width="0.254" layer="16"/>
-<wire x1="50.575084375" y1="85.747859375" x2="52.805653125" y2="83.517290625" width="0.254" layer="16"/>
 <wire x1="35.2552" y1="45.753021875" x2="35.2552" y2="44.958" width="0.254" layer="16"/>
 <wire x1="23.9776" y1="72.463659375" x2="23.9776" y2="57.030621875" width="0.254" layer="16"/>
@@
 <wire x1="29.982159375" y1="80.11921875" x2="29.817059375" y2="80.12175625" width="0.254" layer="16"/>
 <wire x1="29.817059375" y1="80.12175625" x2="28.3845" y2="78.686659375" width="0.254" layer="16"/>
+<wire x1="45.590459375" y1="80.1217625" x2="49.410125" y2="80.1217625" width="0.254" layer="1"/>
+<wire x1="49.410125" y1="80.1217625" x2="52.805653125" y2="83.517290625" width="0.254" layer="1"/>
 </signal>
 <signal name="VMOT">
@@
 <wire x1="50.79491875" y1="68.7857375" x2="50.79491875" y2="80.063340625" width="0.254" layer="16"/>
 <wire x1="32.084840625" y1="118.6943" x2="32.084840625" y2="118.419440625" width="0.254" layer="16"/>
-<wire x1="47.93741875" y1="82.920840625" x2="32.651696875" y2="82.890359375" width="0.254" layer="16"/>
-<wire x1="32.651696875" y1="82.890359375" x2="31.156696875" y2="84.40373125" width="0.254" layer="16"/>
-<wire x1="31.156696875" y1="84.40373125" x2="30.998159375" y2="84.564215625" width="0.254" layer="16"/>
-<wire x1="30.998159375" y1="84.564215625" x2="30.988" y2="84.592159375" width="0.254" layer="16"/>
-<wire x1="50.79491875" y1="80.063340625" x2="47.93741875" y2="82.920840625" width="0.254" layer="16"/>
-<wire x1="31.156696875" y1="84.40373125" x2="30.761940625" y2="84.7984875" width="0.254" layer="16"/>
-<wire x1="30.761940625" y1="84.7984875" x2="30.761940625" y2="118.00331875" width="0.254" layer="16"/>
 <wire x1="30.761940625" y1="118.00331875" x2="31.452921875" y2="118.6943" width="0.254" layer="16"/>
 <wire x1="31.452921875" y1="118.6943" x2="32.084840625" y2="118.6943" width="0.254" layer="16"/>
+<wire x1="30.761940625" y1="100.09631875" x2="30.761940625" y2="118.00331875" width="0.254" layer="16"/>
+<wire x1="50.79491875" y1="80.063340625" x2="30.761940625" y2="100.09631875" width="0.254" layer="16"/>
 </signal>
 <signal name="COMM_2">
@@
 <wire x1="34.89451875" y1="54.099459375" x2="49.837340625" y2="69.04228125" width="0.254" layer="16"/>
 <wire x1="49.837340625" y1="69.04228125" x2="49.837340625" y2="79.1845" width="0.254" layer="16"/>
-<wire x1="47.118271875" y1="81.90356875" x2="24.989790625" y2="81.90356875" width="0.254" layer="16"/>
-<wire x1="49.837340625" y1="79.1845" x2="47.118271875" y2="81.90356875" width="0.254" layer="16"/>
-<wire x1="24.989790625" y1="81.90356875" x2="14.804840625" y2="92.08851875" width="0.254" layer="16"/>
-<wire x1="14.804840625" y1="92.08851875" x2="14.804840625" y2="118.7743" width="0.254" layer="16"/>
+<wire x1="14.804840625" y1="114.217" x2="14.804840625" y2="118.7743" width="0.254" layer="16"/>
+<wire x1="49.837340625" y1="79.1845" x2="14.804840625" y2="114.217" width="0.254" layer="16"/>
 </signal>
 <signal name="N$4">
