File: Eagle/power_multiIO/New folder/task_eagle.brd (EAGLE design)
At the start: 85 x 123.9 mm, 100 parts, among them IC2 ATMEGA640-16AI, IC3 74ACT125D, IC7 FT232RL, IC8 MAX485, K1 G5LE, K2 G5LE, K3 G5LE, K6 G5LE, U1 TC1262-33VDB, U2 Tyco 5-6605758-1, U3 ENC28J60-SSOP, Y2 25MHz

Commit message: rfid and power_multiIO
Routing:
- net VMOT: track 11.6 -> 8.37 mm
- net 12V_IN: track 30.8 -> 30.1 mm

Commit message: small hopper
Parts:
- added ADJUST_OVLO: 200K, SmartPrj:R0603-ROUND
- added ADJUST_UVLO: 250K, SmartPrj:R0603-ROUND
- added C17: 0.47uF, SmartPrj:C0603-ROUND
- added C18: 4.7uF, SmartPrj:C0603-ROUND
- added C21: 0.1uF, SmartPrj:C0603-ROUND
- added PWR-LED1: Amber, SparkFun:LED-0603
- added R15_BYPASS8: 0R, SmartPrj:R0603-ROUND
- added R26, R27: 2.2M, SmartPrj:R0603-ROUND
- added R38: 2.74K, SmartPrj:R0603-ROUND
- added R39, R40, R41: 100K, SmartPrj:R0603-ROUND
- added R42, R43: 10K, SmartPrj:R0603-ROUND
- added U$37: MAX14571, MAX14571:TSSOP14
- added U$38: STPS5L60S, STPS5L60S:SMC
- added U$39: SM6T36CA, ref-packages:DO214AA
- added U$40: NC7WZ07P6X, ref-packages:SC70-6L
- added U$41, U$42: EEV-FK1H331Q, EEVFK1H331Q:EEVFK1H331Q
- moved C12 23.3 mm to (58.5, 88.8), flipped to the bottom
- moved DC2DC_1 18.3 mm to (54.2, 93.5), turned to 0 degrees
- moved D3 16.5 mm to (58.5, 105.1)
- moved PFET-M 16.1 mm to (62.9, 108.3)
- moved K1 14.8 mm to (60.5, 126.2)
- moved K2 14.8 mm to (26.1, 126.2)
- moved K3 14.8 mm to (8.84, 126.3)
- moved K6 14.8 mm to (43.3, 126.2)
- moved U$4 14.8 mm to (80.4, 103.8)
Connections:
- new net 12V_FET: C17.1, D3.C, PFET-M.3, R26.1, R27.1, U$37.IN@1, U$37.IN@2, U$37.IN@3, U$39.C
- new net N$40: PWR-LED1.A, R43.1
- new net N$45: PWR-LED1.C, U$40.5
- new net N$46: R39.1, U$40.2
- new net N$55: R15_BYPASS8.2, U$40.6
- new net OVLO: ADJUST_OVLO.1, R26.2, U$37.OVLO
- new net SETI: R38.1, U$37.SETI
- new net UVLO: ADJUST_UVLO.1, R27.2, U$37.UVLO
- new net XX: R42.2, U$37.FLAG, U$40.1
- net 12V: now also C18.1, U$37.OUT@1, U$37.OUT@2, U$37.OUT@3, U$38.1, U$41.P$2, U$42.P$2; no longer D3.C, PFET-M.3
- net GND: now also ADJUST_OVLO.2, ADJUST_UVLO.2, C17.2, C18.2, C21.2, R38.2, R39.2, R40.1, R41.1, U$37.GND, U$37.HVEN, U$38.2, U$39.A, U$40.3, U$41.P$1, U$42.P$1
- net VCC: now also C21.1, R15_BYPASS8.1, R40.2, R41.2, R42.1, R43.2, U$37.EN, U$37.RIEN, U$40.4
Routing:
- net GND: track 734.5 -> 839.3 mm
- net 12V: track 54.3 -> 123.6 mm, vias 0 -> 2
- net VCC: track 413.6 -> 463.3 mm, vias 22 -> 25
- net 12V_FET: track 0.00 -> 26.4 mm, vias 0 -> 1
- net RELAY_3_IN: track 77.0 -> 92.8 mm
- net RELAY_4_IN: track 85.4 -> 100.3 mm
- net RELAY_2_IN: track 63.5 -> 78.5 mm
- net RELAY_1_IN: track 67.8 -> 82.6 mm, vias 1 -> 3
- net SETI: track 0.00 -> 11.2 mm
- net XX: track 0.00 -> 8.22 mm
- net OVLO: track 0.00 -> 8.01 mm
- net 12V_IN: track 30.1 -> 22.3 mm
- net UVLO: track 0.00 -> 4.16 mm
- net N$55: track 0.00 -> 2.43 mm
- net N$45: track 0.00 -> 2.08 mm
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Other:
- board size 85 x 123.9 mm -> 85 x 140.3 mm
